File: PCB_Rack version/OpenSpritzer2.kicad_pcb (KiCad board)
At the start: 2 copper layers, 180 x 93.8 mm, 32 parts, among them J1 Barrel_Jack, J2 BNC FootPedal, J3 BNC TTL Generator, J4 to Solenoid, SW1 Power Switch, SW2 SW_Push_DPDT, SW3 Rotary Encoder, U1 ESP32-DEVKITC-32D, U2 LM2596S-12, U3 ST7789V Screen

Commit message: Re-update commit
Parts:
- removed NPN (x3): NPN, Package_TO_SOT_THT:TO-92L_Inline_Wide
- removed the REF** at (10.0, 7.50)
- removed the REF** at (161.0, 72.0)
- removed the REF** at (10.0, 72.0)
- removed the REF** at (161.0, 7.50)
- added H1: MountingHole, MountingHole:MountingHole_3mm, F.Cu at (161.0, 7.50)
- added H2: MountingHole, MountingHole:MountingHole_3mm, F.Cu at (161.0, 72.0)
- added H3: MountingHole, MountingHole:MountingHole_3mm, F.Cu at (10.0, 7.50)
- added H4: MountingHole, MountingHole:MountingHole_3mm, F.Cu at (10.0, 72.0)
- added Q1: 2N3904, Package_TO_SOT_THT:TO-92_Inline, F.Cu at (87.5, 65.3)
- added R10: 2kΩ, Resistor_THT:R_Axial_DIN0309_L9.0mm_D3.2mm_P15.24mm_Horizontal, F.Cu at (53.9, 40.0)
- added R11: 1kΩ, Resistor_THT:R_Axial_DIN0309_L9.0mm_D3.2mm_P15.24mm_Horizontal, F.Cu at (53.9, 36.3)
- added R6: 1kΩ, Resistor_THT:R_Axial_DIN0309_L9.0mm_D3.2mm_P15.24mm_Horizontal, F.Cu at (92.8, 61.1)
- added R7: 1MΩ, Resistor_THT:R_Axial_DIN0309_L9.0mm_D3.2mm_P15.24mm_Horizontal, F.Cu at (92.8, 68.6)
- added R8: 2kΩ, Resistor_THT:R_Axial_DIN0309_L9.0mm_D3.2mm_P15.24mm_Horizontal, F.Cu at (92.8, 64.9)
- added R9: 1MΩ, Resistor_THT:R_Axial_DIN0309_L9.0mm_D3.2mm_P15.24mm_Horizontal, F.Cu at (53.9, 43.8)
- moved R3 2.33 mm to (124.7, 56.6)
- moved R4 0.08 mm to (124.7, 52.8)
- moved R5 0.06 mm to (47.5, 65.3)
Connections:
- net GPIO0 renamed Screen_RST
- net GPIO15 renamed Screen_CS
- net GPIO18 renamed Screen_CLK
- net GPIO2 renamed Screen_BL
- net GPIO21 renamed Rotary_SW
- net GPIO23 renamed Screen_DIN
- net GPIO25 renamed Rotary_CLK
- net GPIO26 renamed Rotary_DT
- net GPIO32 renamed Solenoid
- net GPIO34 renamed Pedal
- net GPIO4 renamed Screen_DC
- D4 pad 1: Net-(D4-Pad1) -> GNDREF
- J2 pad 2: VCC 5V -> GNDREF
- R5 pad 2: VCC 5V -> SpritzLED
- U1 pad 11: unconnected-(U1-Pad11) -> TTL_Screen
- U1 pad 29: unconnected-(U1-Pad29) -> TTL
- U1 pad 8: unconnected-(U1-Pad8) -> SpritzLED
Routing:
- net SpritzLED: track 0.00 -> 124.0 mm, vias 0 -> 1
- net Solenoid: track 171.3 -> 66.3 mm, vias 1 -> 0
- net TTL: track 0.00 -> 103.5 mm, vias 0 -> 1
- net TTL_Screen: track 0.00 -> 79.3 mm, vias 0 -> 1
- net VCC 5V: track 360.9 -> 296.7 mm, vias 1 -> 0
- net Net-(D4-Pad1): track 38.0 -> 0.00 mm
- net Net-(R6-Pad1): track 0.00 -> 30.4 mm
- net Net-(R3-Pad1): track 87.5 -> 117.6 mm
- net Net-(J3-Pad1): track 115.0 -> 136.7 mm
- net Net-(R2-Pad2): track 29.5 -> 50.5 mm
- net 3.3V: track 169.6 -> 154.3 mm, vias 0 -> 1
- net Net-(Q1-Pad3): track 8.81 -> 0.00 mm
- net Screen_DIN: track 141.3 -> 136.4 mm
- net Rotary_SW: track 130.5 -> 132.9 mm, vias 1 -> 0
- net Pedal: track 13.7 -> 11.4 mm
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