File: PCB_Rack version/OpenSpritzer2.kicad_sch (KiCad schematic)
At the start: 29 parts, among them J1 Barrel_Jack, J2 BNC FootPedal, J3 BNC TTL Generator, J4 to Solenoid, SW1 Power Switch, SW2 SW_Push_DPDT, SW3 Rotary Encoder, U1 ESP32-DEVKITC-32D, U2 LM2596S-12, U3 ST7789V Screen

Commit message: Re-update commit
Parts:
- removed Q1, Q2, Q3: (no value), symbol Device:Q_NPN_BCE
- added Q1: (no value), symbol Transistor_BJT:2N3904
- added R10, R8: 2kΩ, Resistor_THT:R_Axial_DIN0309_L9.0mm_D3.2mm_P15.24mm_Horizontal, symbol Device:R
- added R11, R6: 1kΩ, Resistor_THT:R_Axial_DIN0309_L9.0mm_D3.2mm_P15.24mm_Horizontal, symbol Device:R
- added R7, R9: (no value), Resistor_THT:R_Axial_DIN0309_L9.0mm_D3.2mm_P15.24mm_Horizontal, symbol Device:R
Connections:
- net GNDREF: now also D4.1 (K), J2.2 (Ext), R10.1, R7.1, R8.1, R9.1
- net VCC 5V: now also Q1.3 (C); no longer J2.2 (Ext), R5.2
- net at J3.1 (In): now also R11.1, R9.2
- net TTL_Screen: now reaches U1.11 (IO27)
- net TTL_Screen: now also R6.2, R7.2
- net TTL: now reaches U1.29 (IO5)
- net TTL: now also R10.2, R11.2
- net SpritzLED: now reaches U1.8 (IO33)
- net SpritzLED: now also R5.2
- net at R2.2, SW2.3 (C): now also Q1.2 (B)
- net GPIO0 renamed Screen_RST
- net GPIO15 renamed Screen_CS
- net GPIO18 renamed Screen_CLK
- net GPIO2 renamed Screen_BL
- net GPIO21 renamed Rotary_SW
- net GPIO23 renamed Screen_DIN
- net GPIO25 renamed Rotary_CLK
- net GPIO26 renamed Rotary_DT
- net GPIO32 renamed Solenoid
- net GPIO34 renamed Pedal
- net GPIO4 renamed Screen_DC
- new net: Q1.1 (E), R6.1, R8.2
Other:
- moved on the sheet: D2, D3, J2, J3, R1, R2, R3, R4, SW2
