File: PCB/OpenSpritzer2.kicad_pcb (KiCad board)
At the start: 2 copper layers, 193.8 x 93.8 mm, 41 parts, among them J1 Barrel_Jack, J2 BNC FootPedal, J3 BNC TTL Generator, J4 to Solenoid, SW1 Power Switch, SW2 SW_Push_DPDT, SW3 Rotary Encoder, U1 ESP32-DEVKITC-32D, U2 LM2596S-12, U3 ST7789V Screen

Commit message: update PCB
Parts:
- removed 10kΩ (x2): 10kΩ, Resistor_THT:R_Axial_DIN0309_L9.0mm_D3.2mm_P15.24mm_Horizontal
- removed 1kΩ (x2): 1kΩ, Resistor_THT:R_Axial_DIN0309_L9.0mm_D3.2mm_P15.24mm_Horizontal
- removed 2kΩ (x2): 2kΩ, Resistor_THT:R_Axial_DIN0309_L9.0mm_D3.2mm_P15.24mm_Horizontal
- removed NPN (x6): NPN, Package_TO_SOT_THT:TO-92L_Inline_Wide
- added C10: 0.1μF, Capacitor_THT:C_Disc_D4.7mm_W2.5mm_P5.00mm, F.Cu at (182.8, 112.7)
- added C11: 100pF, Capacitor_THT:C_Disc_D4.7mm_W2.5mm_P5.00mm, F.Cu at (213.8, 106.7)
- added C12: 22μF, Capacitor_THT:CP_Radial_D6.3mm_P2.50mm, F.Cu at (201.5, 106.4)
- added C13: 100nF, Capacitor_THT:C_Disc_D4.7mm_W2.5mm_P5.00mm, F.Cu at (202.7, 100.5)
- added C14: 100nF, Capacitor_THT:C_Disc_D4.7mm_W2.5mm_P5.00mm, F.Cu at (205.3, 100.5)
- added C15: 0.1μF, Capacitor_THT:C_Disc_D4.7mm_W2.5mm_P5.00mm, F.Cu at (112.3, 138.7)
- added C16: 4.7μF, Capacitor_THT:CP_Radial_D6.3mm_P2.50mm, F.Cu at (115.0, 133.6)
- added C17: 0.1μF, Capacitor_THT:C_Disc_D4.7mm_W2.5mm_P5.00mm, F.Cu at (122.8, 144.8)
- added C18: 10nF, Capacitor_THT:C_Disc_D4.7mm_W2.5mm_P5.00mm, F.Cu at (169.1, 121.2)
- added C19: 10nF, Capacitor_THT:C_Disc_D4.7mm_W2.5mm_P5.00mm, F.Cu at (161.5, 128.3)
- added C20: 0.1μF, Capacitor_THT:C_Disc_D4.7mm_W2.5mm_P5.00mm, F.Cu at (182.8, 125.3)
- added C3: 680μF, Capacitor_THT:CP_Radial_D6.3mm_P2.50mm, F.Cu at (186.6, 56.4)
- added C4: 100μF, Capacitor_THT:CP_Radial_D6.3mm_P2.50mm, F.Cu at (186.6, 60.9)
- added C5: 1μF, Capacitor_THT:C_Disc_D4.7mm_W2.5mm_P5.00mm, F.Cu at (191.5, 60.9)
- added C6: 0.1μF, Capacitor_THT:C_Disc_D4.7mm_W2.5mm_P5.00mm, F.Cu at (191.5, 58.5)
- added C7: 220μF, Capacitor_THT:CP_Radial_D6.3mm_P2.50mm, F.Cu at (217.0, 64.0)
- added C8: 10μF, Capacitor_THT:CP_Radial_D6.3mm_P2.50mm, F.Cu at (108.6, 106.1)
- added C9: 47μF, Capacitor_THT:CP_Radial_D6.3mm_P2.50mm, F.Cu at (108.6, 126.1)
- added D5: 1N4148, Diode_THT:D_DO-35_SOD27_P7.62mm_Horizontal, F.Cu at (225.9, 107.1)
- added D6: Spritz LED, Connector_JST:JST_XH_B2B-XH-A_1x02_P2.50mm_Vertical, F.Cu at (244.0, 122.3)
- added D7: LED Pedal, LED_THT:LED_D3.0mm, F.Cu at (147.5, 145.6)
- added D8: LED TTL, LED_THT:LED_D3.0mm, F.Cu at (129.1, 145.6)
- added F1: Fuse, Maxime:FUSE_65600001009_LTF, F.Cu at (96.8, 96.0)
- added FB1: FerriteBead, Diode_THT:D_5W_P12.70mm_Horizontal, F.Cu at (82.3, 64.5)
- added FB2: FerriteBead, Diode_THT:D_5W_P12.70mm_Horizontal, F.Cu at (113.8, 114.7)
- added J5: BNC TTL, Maxime:BNC_Socket_TYCO-AMP_LargePads, F.Cu at (242.8, 109.0)
- added L2: 2.2μH, Inductor_THT:L_Radial_D6.0mm_P4.00mm, F.Cu at (109.4, 116.1)
- added PS1: IRM-30-24, Converter_ACDC:Converter_ACDC_MeanWell_IRM-10-xx_THT, F.Cu at (88.3, 61.5)
- added Q1: 2N5089, Package_TO_SOT_THT:TO-92L_Inline_Wide, F.Cu at (233.1, 122.3)
- added R10: 47k, Resistor_THT:R_Axial_DIN0309_L9.0mm_D3.2mm_P15.24mm_Horizontal, F.Cu at (248.4, 133.8)
- added R11: 100k, Resistor_THT:R_Axial_DIN0309_L9.0mm_D3.2mm_P15.24mm_Horizontal, F.Cu at (233.2, 129.1)
- added R12: 1k, Resistor_THT:R_Axial_DIN0309_L9.0mm_D3.2mm_P15.24mm_Horizontal, F.Cu at (248.4, 138.5)
- added R13: 10k, Resistor_THT:R_Axial_DIN0309_L9.0mm_D3.2mm_P15.24mm_Horizontal, F.Cu at (165.7, 121.2)
- added R14: 150, Resistor_THT:R_Axial_DIN0309_L9.0mm_D3.2mm_P15.24mm_Horizontal, F.Cu at (161.9, 121.2)
- added R15: 10k, Resistor_THT:R_Axial_DIN0309_L9.0mm_D3.2mm_P15.24mm_Horizontal, F.Cu at (158.2, 128.3)
- added R16: 150, Resistor_THT:R_Axial_DIN0309_L9.0mm_D3.2mm_P15.24mm_Horizontal, F.Cu at (154.4, 128.3)
- added R17: 10k, Resistor_THT:R_Axial_DIN0309_L9.0mm_D3.2mm_P15.24mm_Horizontal, F.Cu at (186.3, 125.3)
- added R18: 150, Resistor_THT:R_Axial_DIN0309_L9.0mm_D3.2mm_P15.24mm_Horizontal, F.Cu at (190.0, 125.3)
- added R19: 220, Resistor_THT:R_Axial_DIN0309_L9.0mm_D3.2mm_P15.24mm_Horizontal, F.Cu at (79.1, 60.0)
- added R20: 1k, Resistor_THT:R_Axial_DIN0309_L9.0mm_D3.2mm_P15.24mm_Horizontal, F.Cu at (150.1, 134.6)
- added R21: 1k, Resistor_THT:R_Axial_DIN0309_L9.0mm_D3.2mm_P15.24mm_Horizontal, F.Cu at (129.1, 134.6)
- added R22: 100, Resistor_THT:R_Axial_DIN0309_L9.0mm_D3.2mm_P15.24mm_Horizontal, F.Cu at (137.5, 119.4)
- added R23: 100, Resistor_THT:R_Axial_DIN0309_L9.0mm_D3.2mm_P15.24mm_Horizontal, F.Cu at (141.7, 119.4)
- added R24: 10k, Resistor_THT:R_Axial_DIN0309_L9.0mm_D3.2mm_P15.24mm_Horizontal, F.Cu at (133.3, 119.4)
- added R25: 10k, Resistor_THT:R_Axial_DIN0309_L9.0mm_D3.2mm_P15.24mm_Horizontal, F.Cu at (145.9, 119.4)
- added R6: 4.7k, Resistor_THT:R_Axial_DIN0309_L9.0mm_D3.2mm_P15.24mm_Horizontal, F.Cu at (198.6, 113.2)
- added R7: 10k, Resistor_THT:R_Axial_DIN0309_L9.0mm_D3.2mm_P15.24mm_Horizontal, F.Cu at (194.7, 115.3)
- added R8: 22, Resistor_THT:R_Axial_DIN0309_L9.0mm_D3.2mm_P15.24mm_Horizontal, F.Cu at (188.0, 67.5)
- added R9: 22, Resistor_THT:R_Axial_DIN0309_L9.0mm_D3.2mm_P15.24mm_Horizontal, F.Cu at (183.3, 67.5)
- added RV1: Varistor, Capacitor_THT:C_Disc_D11.0mm_W5.0mm_P5.00mm, F.Cu at (119.9, 105.9)
- added TH1: Thermistor_NTC, Capacitor_THT:C_Disc_D11.0mm_W5.0mm_P5.00mm, F.Cu at (127.5, 105.9)
- added U4: ESP32-DEVKITC-32D, Maxime:MODULE_ESP32-DEVKITC-32D, F.Cu at (222.5, 84.5)
- added U5: ST7789V Screen, Connector_JST:JST_XH_B8B-XH-A_1x08_P2.50mm_Vertical, F.Cu at (121.3, 138.8)
- C1: value 680μF -> 470μF
- C2: value 220μF -> 0.1μF; footprint Capacitor_THT:CP_Radial_D6.3mm_P2.50mm -> Capacitor_THT:C_Disc_D4.7mm_W2.5mm_P5.00mm
- D1: value 1N5822 -> SMBJ33A; footprint Diode_THT:D_DO-201AD_P15.24mm_Horizontal -> PCM_JLCPCB:D_SMB
- D2: value LED Pedal -> P6SKE6.8A; footprint LED_THT:LED_D3.0mm -> PCM_JLCPCB:D_SMB
- D3: value LED TTL -> 1N5822; footprint LED_THT:LED_D3.0mm -> Diode_THT:D_DO-201AD_P15.24mm_Horizontal
- D4: value Spritz LED -> SMAJ5.0A; footprint Connector_JST:JST_XH_B2B-XH-A_1x02_P2.50mm_Vertical -> Diode_SMD:D_SMA
- J1: value Barrel_Jack -> Screw_Terminal; footprint Connector_BarrelJack:BarrelJack_Horizontal -> TerminalBlock_Phoenix:TerminalBlock_Phoenix_MKDS-1,5-2-5.08_1x02_P5.08mm_Horizontal
- J2: value BNC FootPedal -> Screw_Terminal; footprint Maxime:BNC_Socket_TYCO-AMP_LargePads -> TerminalBlock_Phoenix:TerminalBlock_Phoenix_MKDS-1,5-2-5.08_1x02_P5.08mm_Horizontal
- J3: value BNC TTL Generator -> to Solenoid; footprint Maxime:BNC_Socket_TYCO-AMP_LargePads -> Connector_JST:JST_XH_B3B-XH-A_1x03_P2.50mm_Vertical
- J4: value to Solenoid -> BNC Pedal; footprint Connector_JST:JST_XH_B3B-XH-A_1x03_P2.50mm_Vertical -> Maxime:BNC_Socket_TYCO-AMP_LargePads
- R1: value 220Ω -> 1k
- R2: value 220Ω -> 100k
- R3: value 1kΩ -> 100
- R4: value 2kΩ -> 10k
- R5: value 220Ω -> 470
- SW1: value Power Switch -> SW_SPST_LED; footprint Connector_JST:JST_XH_B3B-XH-A_1x03_P2.50mm_Vertical -> TerminalBlock_Phoenix:TerminalBlock_Phoenix_MKDS-1,5-3-5.08_1x03_P5.08mm_Horizontal
- SW2: value SW_Push_DPDT -> Rotary Encoder; footprint Maxime:maxi_DPDT_Angled -> Connector_PinHeader_2.54mm:PinHeader_1x05_P2.54mm_Vertical
- SW3: value Rotary Encoder -> SW_Push_DPDT; footprint Connector_PinHeader_2.54mm:PinHeader_1x05_P2.54mm_Vertical -> Maxime:maxi_DPDT_Angled
- U1: value ESP32-DEVKITC-32D -> LM2596T-3.3; footprint Module:MODULE_ESP32-DEVKITC-32D -> Package_TO_SOT_THT:TO-220-5_P3.4x3.7mm_StaggerOdd_Lead3.8mm_Vertical
- U2: value LM2596S-12 -> SN74HC14N; footprint Package_TO_SOT_THT:TO-220-5_P3.4x3.7mm_StaggerOdd_Lead3.8mm_Vertical -> Package_DIP:DIP-14_W7.62mm_Socket_LongPads
- U3: value ST7789V Screen -> VO615A; footprint Connector_JST:JST_XH_B8B-XH-A_1x08_P2.50mm_Vertical -> Package_DIP:DIP-4_W7.62mm_Socket_LongPads
- moved U3 176.2 mm to (217.4, 110.9)
- moved D4 162.7 mm to (231.0, 112.2), turned to 180 degrees
- moved J3 148.5 mm to (53.5, 53.2), turned to 0 degrees
- moved J4 137.9 mm to (242.8, 60.0), turned to -90 degrees
- moved R5 137.4 mm to (218.2, 103.0), turned to 0 degrees
- moved H3 127.4 mm to (55.0, 145.0)
- moved D3 126.2 mm to (207.0, 54.8)
- moved J2 115.4 mm to (86.0, 96.0), turned to 0 degrees
- moved REF** 102.9 mm to (57.3, 122.3), turned to 90 degrees
- moved ? 95.0 mm to (92.7, 109.0)
- moved U2 90.9 mm to (172.1, 112.7)
- moved C1 86.9 mm to (69.7, 52.7), turned to -90 degrees
- moved REF** 86.7 mm to (75.3, 122.3), turned to 180 degrees
- moved L1 83.0 mm to (207.0, 62.0), turned to -90 degrees
- moved SW1 80.1 mm to (141.0, 96.0)
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Connections:
- C1 pad 1: Vin 24V -> +24V
- C2 pad 1: VCC 5V -> +24V
- D1 pad 1: Net-(D1-K) -> +24V
- D2 pad 1: GNDREF -> Solenoid
- D2 pad 2: Net-(D2-A) -> GNDREF
- D3 pad 1: GNDREF -> Net-(D3-K)
- D3 pad 2: Net-(D3-A) -> GNDREF
- D4 pad 1: Net-(D4-K) -> Net-(D4-A1)
- D4 pad 2: Net-(D4-A) -> Net-(D4-A2)
- H1 pad : (no net) -> Earth_Protective
- H2 pad : (no net) -> Earth_Protective
- H3 pad : (no net) -> Earth_Protective
- H4 pad : (no net) -> Earth_Protective
- J1 pad 1: Net-(J1-Pad1) -> Net-(J1-Pin_1)
- J1 pad 2: GNDREF -> AC/N
- J2 pad 1: Net-(J2-In) -> Earth_Protective
- J3 pad 1: Net-(J3-In) -> GNDREF
- J3 pad 2: GNDREF -> +24V
- J4 pad 1: GNDREF -> Net-(J4-In)
- J4 pad 2: Vin 24V -> Pedal_Input
- L1 pad 1: Net-(D1-K) -> Net-(D3-K)
- L1 pad 2: VCC 5V -> Net-(U1-FB)
- R1 pad 1: Net-(D2-A) -> AC/N
- R1 pad 2: Net-(R1-Pad2) -> Net-(SW1-K)
- R2 pad 1: Net-(D3-A) -> Solenoid
- R2 pad 2: Net-(Q1-B) -> GNDREF
- R3 pad 1: Net-(R3-Pad1) -> Net-(J4-In)
- R3 pad 2: GPIO34 -> 3.3V
- R4 pad 1: GNDREF -> Pedal_Input
- R4 pad 2: GPIO34 -> GNDREF
- R5 pad 1: Net-(D4-A) -> Net-(D5-K)
- R5 pad 2: VCC 5V -> Net-(D4-A1)
- REF** pad : (no net) -> Earth_Protective (x2)
- SW1 pad 1: Net-(J1-Pad1) -> Net-(F1-Pad2)
- SW1 pad 2: Vin 24V -> Net-(SW1-A)
- SW1 pad 3: GNDREF -> Net-(SW1-K)
- SW2 pad 1: Net-(R1-Pad2) -> RotEn_CLK
- SW2 pad 2: VCC 5V -> RotEn_DT
- SW2 pad 3: Net-(Q1-B) -> RotEn_SW
- SW2 pad 4: Net-(J2-In) -> 3.3V
- SW2 pad 5: Net-(R3-Pad1) -> GNDREF
- SW3 pad 1: GPIO25 -> ESP_En
- SW3 pad 2: GPIO26 -> Net-(R19-Pad1)
- SW3 pad 3: GPIO21 -> TTL_En
- SW3 pad 4: 3.3V -> Net-(R20-Pad2)
- SW3 pad 5: GNDREF -> 3.3V
- U1 pad 1: 3.3V -> +24V
- U1 pad 2: unconnected-(U1-EN-Pad2) -> Net-(D3-K)
- U1 pad 3: unconnected-(U1-SENSOR_VP-Pad3) -> GNDREF
- U1 pad 4: unconnected-(U1-SENSOR_VN-Pad4) -> Net-(U1-FB)
- U1 pad 5: GPIO34 -> GNDREF
- U2 pad 1: Vin 24V -> Net-(C11-Pad1)
- U2 pad 2: Net-(D1-K) -> TTL_En
- U2 pad 3: GNDREF -> Net-(C18-Pad1)
- U2 pad 4: VCC 5V -> Rot_CLK
- U2 pad 5: GNDREF -> Net-(C19-Pad1)
- U3 pad 1: 3.3V -> Net-(D5-K)
- U3 pad 2: GNDREF -> Net-(D4-A2)
- U3 pad 3: GPIO23 -> GNDREF
- U3 pad 4: GPIO18 -> Net-(C11-Pad1)
Routing:
- net Earth_Protective: track 0.00 -> 442.0 mm, vias 0 -> 5
- net Net-(J3-In): track 353.2 -> 0.00 mm
- net GPIO21: track 292.9 -> 0.00 mm
- net VCC 5V: track 284.2 -> 0.00 mm
- net Solenoid: track 0.00 -> 258.4 mm, vias 0 -> 2
- net 3.3V: track 175.6 -> 428.4 mm, vias 0 -> 2
- net GPIO33: track 204.5 -> 0.00 mm
- net GPIO26: track 197.6 -> 0.00 mm
- net GPIO25: track 193.8 -> 0.00 mm
- net ESP_En: track 0.00 -> 191.1 mm
- net GPIO15: track 175.9 -> 0.00 mm
- net GPIO4: track 163.6 -> 0.00 mm
- net GPIO0: track 162.6 -> 0.00 mm
- net +24V: track 0.00 -> 162.4 mm
- net GPIO2: track 162.3 -> 0.00 mm
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Other:
- board size 193.8 x 93.8 mm -> 200 x 100 mm
- board text added: "+"
- board text added: "-"
- board text added: "0215001.MXP"
- board text added: "220V"
- board text added: "2743003112"
- board text added: "2743009112"
- board text added: "AC/DC CONVERTER 24V 1.3A IRM-30-24"
- board text added: "AC/L"
- board text added: "AC/N"
- board text added: "B57236S0100M000"
- board text added: "B72214S0271K101"
- board text added: "IEC Inlet Filter TE 6609015-3"
- board text added: "OpenSpritzer v2.3"
- board text added: "Protective Earth"
- board text added: "S"
- board text added: "Solenoid Festo MHJ10-S-2,5-QS-6-HF"
- board text removed: "24V in"
- board text removed: "3.3v"
- board text removed: "CLK"
- board text removed: "DT"
- board text removed: "GND"
- board text removed: "OpenSpritzer v2.2"
- board text removed: "SW"
- board text removed: "Solenoid Festo - MHJ10-S-2,5-QS-6-HF"
- board text removed: "by MJY Zimmermann"
