File: PCB/OpenSpritzer2.kicad_sch (KiCad schematic)
At the start: 79 parts, among them J1 Screw_Terminal, J2 Screw_Terminal, J3 to Solenoid, J4 BNC Pedal, J5 BNC TTL, Q1 2N5089, SW1 SW_SPST_LED, SW2 Rotary Encoder, SW3 SW_Push_DPDT, U1 LM2596T-3.3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

Commit message: update PCB
Parts:
- C10, C15, C17, C2, C20, C6: value 100nF -> 0.1μF
- C5: value 1uF -> 1μF
Changed lines of the file:
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@@
 			)
 		)
-		(property "Value" "100nF"
+		(property "Value" "0.1μF"
 			(at 36.195 43.18 0)
 			(effects
@@
 			)
 		)
-		(property "Value" "100nF"
+		(property "Value" "0.1μF"
 			(at 262.89 141.605 0)
 			(effects
@@
 			)
 		)
-		(property "Value" "100nF"
+		(property "Value" "0.1μF"
 			(at 41.91 98.425 90)
 			(effects
@@
 			)
 		)
-		(property "Value" "100nF"
+		(property "Value" "0.1μF"
 			(at 40.64 71.755 0)
 			(effects
@@
 			)
 		)
-		(property "Value" "100nF"
+		(property "Value" "0.1μF"
 			(at 267.97 69.215 0)
 			(effects
@@
 			)
 		)
-		(property "Value" "1uF"
+		(property "Value" "1μF"
 			(at 35.56 74.295 0)
 			(effects
@@
 			)
 		)
-		(property "Value" "100nF"
+		(property "Value" "0.1μF"
 			(at 253.365 102.87 0)
 			(effects
